File: wind_sensor.kicad_pcb (KiCad board)
At the start: 2 copper layers, 13 parts, among them J1 Conn_01x08_Male, J2 Conn_01x08_Male, U1 AS5600, U2 MAX40200AUK

Commit message: remove regulator
Parts:
- moved J2 95.0 mm to (73.4, 114.3), turned to 180 degrees
- moved J1 79.0 mm to (52.1, 97.0)
Changed lines of the file:
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@@
   )
   (footprint "Connector_PinHeader_2.54mm:PinHeader_1x08_P2.54mm_Vertical" (layer "F.Cu")
-    (at 64.67 19.065)
+    (at 52.07 97.028)
     (descr "Through hole straight pin header, 1x08, 2.54mm pitch, single row")
     (tags "Through hole pin header THT 1x08 2.54mm single row")
@@
   )
   (footprint "Connector_PinHeader_2.54mm:PinHeader_1x08_P2.54mm_Vertical" (layer "F.Cu")
-    (at 72.39 19.2775)
+    (at 73.406 114.3 180)
     (descr "Through hole straight pin header, 1x08, 2.54mm pitch, single row")
     (tags "Through hole pin header THT 1x08 2.54mm single row")
@@
     (fp_line (start 1.27 19.05) (end -1.27 19.05) (layer "F.Fab") (width 0.1))
     (fp_line (start -0.635 -1.27) (end 1.27 -1.27) (layer "F.Fab") (width 0.1))
-    (pad "1" thru_hole rect (at 0 0) (size 1.7 1.7) (drill 1) (layers *.Cu *.Mask)
+    (pad "1" thru_hole rect (at 0 0 180) (size 1.7 1.7) (drill 1) (layers *.Cu *.Mask)
       (net 18 "/PWM") (pinfunction "Pin_1") (pintype "passive"))
-    (pad "2" thru_hole oval (at 0 2.54) (size 1.7 1.7) (drill 1) (layers *.Cu *.Mask)
+    (pad "2" thru_hole oval (at 0 2.54 180) (size 1.7 1.7) (drill 1) (layers *.Cu *.Mask)
       (net 19 "/INT") (pinfunction "Pin_2") (pintype "passive"))
-    (pad "3" thru_hole oval (at 0 5.08) (size 1.7 1.7) (drill 1) (layers *.Cu *.Mask)
+    (pad "3" thru_hole oval (at 0 5.08 180) (size 1.7 1.7) (drill 1) (layers *.Cu *.Mask)
       (net 20 "/TX") (pinfunction "Pin_3") (pintype "passive"))
-    (pad "4" thru_hole oval (at 0 7.62) (size 1.7 1.7) (drill 1) (layers *.Cu *.Mask)
+    (pad "4" thru_hole oval (at 0 7.62 180) (size 1.7 1.7) (drill 1) (layers *.Cu *.Mask)
       (net 21 "/RX") (pinfunction "Pin_4") (pintype "passive"))
-    (pad "5" thru_hole oval (at 0 10.16) (size 1.7 1.7) (drill 1) (layers *.Cu *.Mask)
+    (pad "5" thru_hole oval (at 0 10.16 180) (size 1.7 1.7) (drill 1) (layers *.Cu *.Mask)
       (net 8 "/SCL") (pinfunction "Pin_5") (pintype "passive"))
-    (pad "6" thru_hole oval (at 0 12.7) (size 1.7 1.7) (drill 1) (layers *.Cu *.Mask)
+    (pad "6" thru_hole oval (at 0 12.7 180) (size 1.7 1.7) (drill 1) (layers *.Cu *.Mask)
       (net 9 "/SDA") (pinfunction "Pin_6") (pintype "passive"))
-    (pad "7" thru_hole oval (at 0 15.24) (size 1.7 1.7) (drill 1) (layers *.Cu *.Mask)
+    (pad "7" thru_hole oval (at 0 15.24 180) (size 1.7 1.7) (drill 1) (layers *.Cu *.Mask)
       (net 22 "/5V") (pinfunction "Pin_7") (pintype "passive"))
-    (pad "8" thru_hole oval (at 0 17.78) (size 1.7 1.7) (drill 1) (layers *.Cu *.Mask)
+    (pad "8" thru_hole oval (at 0 17.78 180) (size 1.7 1.7) (drill 1) (layers *.Cu *.Mask)
       (net 2 "GND") (pinfunction "Pin_8") (pintype "passive"))
     (model "${KICAD6_3DMODEL_DIR}/Connector_PinHeader_2.54mm.3dshapes/PinHeader_1x08_P2.54mm_Vertical.wrl"
@@
     )
   )
+  (gr_rect (start 50.8 75.438) (end 75.946 121.412) (layer "F.Cu") (width 0.2) (fill none))
 )

Commit message: Update wind_sensor.kicad_pcb
Parts:
- removed R5: 10k, Resistor_THT:R_Array_SIP4
- removed U2: MAX40200AUK, Package_TO_SOT_SMD:SOT-23-5
- moved R4 91.9 mm to (57.9, 87.9)
- moved R6 82.6 mm to (63.0, 87.7), turned to -90 degrees
- moved U1 79.7 mm to (63.0, 79.0)
- moved C1 78.4 mm to (71.6, 79.5)
- moved C2 76.7 mm to (54.4, 80.0)
- moved R3 73.8 mm to (72.1, 88.9)
- moved R1 71.2 mm to (61.5, 94.0)
- moved R2 67.8 mm to (68.1, 87.0)
- moved LD1 63.0 mm to (53.8, 95.8), turned to 90 degrees
- moved J2 4.89 mm to (74.2, 119.1)
- moved J1 4.83 mm to (52.3, 101.9)
